Commit message: fastsam sim integration

File: panther_gazebo/urdf/asus_camera.urdf.xacro (robot description, xacro)
@@ -79,9 +79,10 @@
           <update_rate>60</update_rate>
           <camera>
-            <horizontal_fov>${60 * M_PI/180.0}</horizontal_fov>
+            <horizontal_fov>${76 * M_PI/180.0}</horizontal_fov>
+            <vertical_fov>${47 * M_PI/180.0}</vertical_fov>
             <image>
               <format>R8G8B8</format>
-              <width>120</width> <!-- 120, 90 //320, 240 // 480, 480 -->
-              <height>120</height> <!--Note that the focal length is given by f = (width/2) / tan( horizontal_fov/2)
+              <width>480</width> <!-- 120, 90 //320, 240 // 480, 480 -->
+              <height>480</height> <!--Note that the focal length is given by f = (width/2) / tan( horizontal_fov/2)
                                                      vertical_fov is given by 2*arctan(height/(2*f))
                                                     Also, the camera_info msg will have:

File: panther_gazebo/urdf/quadrotor_with_asus.urdf.xacro (robot description, xacro)
@@ -9,6 +9,7 @@
     <xacro:include filename="$(find panther_gazebo)/urdf/asus_camera.urdf.xacro" />
     <xacro:asus_camera name="camera" parent="base_link">
-     <!-- <origin xyz="0.1 0.0 -0.03" rpy="0 0 0"/>-->
-         <origin xyz="0.1 0.0 0" rpy="0 0.0 0"/>  <!-- 0 -0.78 0 -->
+        <!-- <origin xyz="0.1 0.0 -0.03" rpy="0 0 0"/>-->
+        <!-- <origin xyz="0.1 0.0 0" rpy="0 0.0 0"/> -->  <!-- 0 -0.78 0 -->
+        <origin xyz="0 0 -0.2" rpy="0 ${M_PI/2} 0"/>  <!-- 0 -0.78 0 -->
     </xacro:asus_camera>
        <!-- Sonar height sensor -->

Commit message: forward facing camera fix

File: panther_gazebo/urdf/asus_camera.urdf.xacro (robot description, xacro)
@@ -79,10 +79,9 @@
           <update_rate>60</update_rate>
           <camera>
-            <horizontal_fov>${76 * M_PI/180.0}</horizontal_fov>
-            <vertical_fov>${47 * M_PI/180.0}</vertical_fov>
+            <horizontal_fov>${60 * M_PI/180.0}</horizontal_fov>
             <image>
               <format>R8G8B8</format>
-              <width>480</width> <!-- 120, 90 //320, 240 // 480, 480 -->
-              <height>480</height> <!--Note that the focal length is given by f = (width/2) / tan( horizontal_fov/2)
+              <width>120</width> <!-- 120, 90 //320, 240 // 480, 480 -->
+              <height>120</height> <!--Note that the focal length is given by f = (width/2) / tan( horizontal_fov/2)
                                                      vertical_fov is given by 2*arctan(height/(2*f))
                                                     Also, the camera_info msg will have:

File: panther_gazebo/urdf/quadrotor_with_asus.urdf.xacro (robot description, xacro)
@@ -9,7 +9,6 @@
     <xacro:include filename="$(find panther_gazebo)/urdf/asus_camera.urdf.xacro" />
     <xacro:asus_camera name="camera" parent="base_link">
-        <!-- <origin xyz="0.1 0.0 -0.03" rpy="0 0 0"/>-->
-        <!-- <origin xyz="0.1 0.0 0" rpy="0 0.0 0"/> -->  <!-- 0 -0.78 0 -->
-        <origin xyz="0 0 -0.2" rpy="0 ${M_PI/2} 0"/>  <!-- 0 -0.78 0 -->
+     <!-- <origin xyz="0.1 0.0 -0.03" rpy="0 0 0"/>-->
+         <origin xyz="0.1 0.0 0" rpy="0 0.0 0"/>  <!-- 0 -0.78 0 -->
     </xacro:asus_camera>
        <!-- Sonar height sensor -->
